Commit message: Update roam.urdf
changed mesh paths to work on all systems

File: catkin_ws/src/roam_description/urdf/roam.urdf (robot description, URDF)
Before this commit: robot roam, 17 links, 16 joints
Links:
- link link_1: geometry collision box size=0.126 0.08 0.121; visual mesh filename=package://roam_description/meshes/link_1.dae
- link link_2: geometry collision box size=0.04 0.08 0.319; visual mesh filename=package://roam_description/meshes/link_2.dae
- link link_3: geometry collision box size=0.124 0.074 0.213; visual mesh filename=package://roam_description/meshes/link_3.dae
- link link_4: geometry collision box size=0.055 0.222 0.073; visual mesh filename=package://roam_description/meshes/link_4.dae
- link ratrig_link: geometry collision box size=0.037 0.140 0.537; visual mesh filename=package://roam_description/meshes/ratrig.dae
